File: projects/RoboRio/RoboRioExpansionBoard/partsFound.sch (EAGLE design)
At the start: 4 parts, among them IC1 LM1086

Commit message: more parts in partsFound
Forgot to save it last time.
Parts:
- added IC2: 24LC256P, microchip:24LC256P
- added IC3: 40109, 40xx-2:40109
- added LED1, LED2, LED3: (no value), led:LED3MM
- added Q1: (no value), crystal:CRYSTALHC49U70
- added R1: (no value), resistor:R-US_0207/7
Changed lines of the file:
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@@
 <part name="IC1" library="oli" deviceset="LM1086*" device=""/>
 <part name="U$2" library="parallax_propeller (1)" deviceset="P8X32A-D40" device=""/>
+<part name="Q1" library="crystal" deviceset="CRYSTAL" device="HC49U70"/>
+<part name="IC2" library="microchip" deviceset="24*" device="P" technology="LC256"/>
+<part name="LED1" library="led" deviceset="LED" device="3MM"/>
+<part name="LED2" library="led" deviceset="LED" device="3MM"/>
+<part name="LED3" library="led" deviceset="LED" device="3MM"/>
+<part name="R1" library="resistor" deviceset="R-US_" device="0207/7"/>
+<part name="IC3" library="40xx-2" deviceset="40109" device=""/>
 </parts>
 <sheets>
@@
 <instance part="IC1" gate="G$1" x="83.82" y="114.3"/>
 <instance part="U$2" gate="P8X32A-D40" x="45.72" y="35.56"/>
+<instance part="Q1" gate="G$1" x="38.1" y="-7.62"/>
+<instance part="IC2" gate="G$1" x="43.18" y="-27.94"/>
+<instance part="LED1" gate="G$1" x="35.56" y="-48.26" rot="R90"/>
+<instance part="LED2" gate="G$1" x="45.72" y="-48.26" rot="R90"/>
+<instance part="LED3" gate="G$1" x="55.88" y="-48.26" rot="R90"/>
+<instance part="R1" gate="G$1" x="38.1" y="-58.42" rot="R180"/>
+<instance part="IC3" gate="A" x="45.72" y="-71.12"/>
+<instance part="IC3" gate="B" x="76.2" y="-71.12"/>
+<instance part="IC3" gate="C" x="106.68" y="-71.12"/>
+<instance part="IC3" gate="D" x="134.62" y="-71.12"/>
 </instances>
 <busses>
