File: projects/RoboRio/RoboRioExpansionBoard/ExpansionBoardV1.sch (EAGLE design)
At the start: 37 parts, among them IC1 MCP3008, IC2 40109, Q1 5MHz

Commit message: Updated resistor to the correct package
The I2C pullup for the eeprom
How can we only have one resistor?
Parts:
- R1: device resistor:R-US_0207/7 -> resistor:R-US_0309/V
Changed lines of the file:
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@@
 <grid distance="0.1" unitdist="inch" unit="inch" style="lines" multiple="1" display="no" altdistance="0.01" altunitdist="inch" altunit="inch"/>
 <layers>
-<layer number="1" name="Top" color="4" fill="1" visible="yes" active="no"/>
-<layer number="16" name="Bottom" color="1" fill="1" visible="yes" active="no"/>
-<layer number="17" name="Pads" color="2" fill="1" visible="yes" active="no"/>
-<layer number="18" name="Vias" color="2" fill="1" visible="yes" active="no"/>
-<layer number="19" name="Unrouted" color="6" fill="1" visible="yes" active="no"/>
-<layer number="20" name="Dimension" color="15" fill="1" visible="yes" active="no"/>
-<layer number="21" name="tPlace" color="7" fill="1" visible="yes" active="no"/>
-<layer number="22" name="bPlace" color="7" fill="1" visible="yes" active="no"/>
-<layer number="23" name="tOrigins" color="15" fill="1" visible="yes" active="no"/>
-<layer number="24" name="bOrigins" color="15" fill="1" visible="yes" active="no"/>
-<layer number="25" name="tNames" color="7" fill="1" visible="yes" active="no"/>
-<layer number="26" name="bNames" color="7" fill="1" visible="yes" active="no"/>
-<layer number="27" name="tValues" color="7" fill="1" visible="yes" active="no"/>
-<layer number="28" name="bValues" color="7" fill="1" visible="yes" active="no"/>
+<layer number="1" name="Top" color="4" fill="1" visible="no" active="no"/>
+<layer number="16" name="Bottom" color="1" fill="1" visible="no" active="no"/>
+<layer number="17" name="Pads" color="2" fill="1" visible="no" active="no"/>
+<layer number="18" name="Vias" color="2" fill="1" visible="no" active="no"/>
+<layer number="19" name="Unrouted" color="6" fill="1" visible="no" active="no"/>
+<layer number="20" name="Dimension" color="15" fill="1" visible="no" active="no"/>
+<layer number="21" name="tPlace" color="7" fill="1" visible="no" active="no"/>
+<layer number="22" name="bPlace" color="7" fill="1" visible="no" active="no"/>
+<layer number="23" name="tOrigins" color="15" fill="1" visible="no" active="no"/>
+<layer number="24" name="bOrigins" color="15" fill="1" visible="no" active="no"/>
+<layer number="25" name="tNames" color="7" fill="1" visible="no" active="no"/>
+<layer number="26" name="bNames" color="7" fill="1" visible="no" active="no"/>
+<layer number="27" name="tValues" color="7" fill="1" visible="no" active="no"/>
+<layer number="28" name="bValues" color="7" fill="1" visible="no" active="no"/>
 <layer number="29" name="tStop" color="7" fill="3" visible="no" active="no"/>
 <layer number="30" name="bStop" color="7" fill="6" visible="no" active="no"/>
@@
 <layer number="35" name="tGlue" color="7" fill="4" visible="no" active="no"/>
 <layer number="36" name="bGlue" color="7" fill="5" visible="no" active="no"/>
-<layer number="37" name="tTest" color="7" fill="1" visible="yes" active="no"/>
-<layer number="38" name="bTest" color="7" fill="1" visible="yes" active="no"/>
+<layer number="37" name="tTest" color="7" fill="1" visible="no" active="no"/>
+<layer number="38" name="bTest" color="7" fill="1" visible="no" active="no"/>
 <layer number="39" name="tKeepout" color="4" fill="11" visible="no" active="no"/>
 <layer number="40" name="bKeepout" color="1" fill="11" visible="no" active="no"/>
@@
 <layer number="44" name="Drills" color="7" fill="1" visible="no" active="no"/>
 <layer number="45" name="Holes" color="7" fill="1" visible="no" active="no"/>
-<layer number="46" name="Milling" color="3" fill="1" visible="yes" active="no"/>
-<layer number="47" name="Measures" color="7" fill="1" visible="yes" active="no"/>
-<layer number="48" name="Document" color="7" fill="1" visible="yes" active="no"/>
-<layer number="49" name="Reference" color="7" fill="1" visible="yes" active="no"/>
-<layer number="50" name="dxf" color="7" fill="1" visible="yes" active="no"/>
-<layer number="51" name="tDocu" color="7" fill="1" visible="yes" active="no"/>
-<layer number="52" name="bDocu" color="7" fill="1" visible="yes" active="no"/>
-<layer number="53" name="tGND_GNDA" color="7" fill="9" visible="yes" active="no"/>
-<layer number="54" name="bGND_GNDA" color="1" fill="9" visible="yes" active="no"/>
-<layer number="56" name="wert" color="7" fill="1" visible="yes" active="no"/>
-<layer number="57" name="tCAD" color="7" fill="1" visible="yes" active="no"/>
+<layer number="46" name="Milling" color="3" fill="1" visible="no" active="no"/>
+<layer number="47" name="Measures" color="7" fill="1" visible="no" active="no"/>
+<layer number="48" name="Document" color="7" fill="1" visible="no" active="no"/>
+<layer number="49" name="Reference" color="7" fill="1" visible="no" active="no"/>
+<layer number="50" name="dxf" color="7" fill="1" visible="no" active="no"/>
+<layer number="51" name="tDocu" color="7" fill="1" visible="no" active="no"/>
+<layer number="52" name="bDocu" color="7" fill="1" visible="no" active="no"/>
+<layer number="53" name="tGND_GNDA" color="7" fill="9" visible="no" active="no"/>
+<layer number="54" name="bGND_GNDA" color="1" fill="9" visible="no" active="no"/>
+<layer number="56" name="wert" color="7" fill="1" visible="no" active="no"/>
+<layer number="57" name="tCAD" color="7" fill="1" visible="no" active="no"/>
 <layer number="90" name="Modules" color="5" fill="1" visible="yes" active="yes"/>
 <layer number="91" name="Nets" color="2" fill="1" visible="yes" active="yes"/>
@@
 <part name="+3V1" library="supply1" deviceset="+3V3" device=""/>
 <part name="+3V2" library="supply1" deviceset="+3V3" device=""/>
-<part name="R1" library="resistor" deviceset="R-US_" device="0207/7" value="10k"/>
+<part name="R1" library="resistor" deviceset="R-US_" device="0309/V" value="10k"/>
 <part name="U$3" library="PropPlug" deviceset="PROP_PLUG" device=""/>
 <part name="GND4" library="supply1" deviceset="GND" device=""/>

Commit message: Added some beautiful resistors to the status LEDs
your welcome!
Parts:
- added R2, R3, R4: 10k, resistor:R-US_0309/V
Connections:
- new net N$12: R2.1, YELLOW.K
- new net N$13: R3.1, RED.K
- new net N$14: GREEN.K, R4.2
- net IO4: now also R2.2, R4.1; no longer GREEN.K
- net IO5: no longer YELLOW.K
- net IO6: now also R3.2; no longer RED.K
Other:
- moved on the sheet: GREEN, RED, YELLOW
Changed lines of the file:
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@@
 <part name="+3V6" library="supply1" deviceset="+3V3" device=""/>
 <part name="+3V7" library="supply1" deviceset="+3V3" device=""/>
+<part name="R2" library="resistor" deviceset="R-US_" device="0309/V" value="10k"/>
+<part name="R3" library="resistor" deviceset="R-US_" device="0309/V" value="10k"/>
+<part name="R4" library="resistor" deviceset="R-US_" device="0309/V" value="10k"/>
 </parts>
 <sheets>
@@
 <instance part="GND7" gate="1" x="78.74" y="114.3"/>
 <instance part="+3V5" gate="G$1" x="81.28" y="109.22" rot="R90"/>
-<instance part="GREEN" gate="A" x="17.78" y="185.42" rot="R270"/>
-<instance part="YELLOW" gate="A" x="17.78" y="195.58" rot="R270"/>
-<instance part="RED" gate="A" x="17.78" y="205.74" rot="R270"/>
-<instance part="GND10" gate="1" x="30.48" y="182.88"/>
+<instance part="GREEN" gate="A" x="22.86" y="185.42" rot="R270"/>
+<instance part="YELLOW" gate="A" x="22.86" y="195.58" rot="R270"/>
+<instance part="RED" gate="A" x="22.86" y="205.74" rot="R270"/>
+<instance part="GND10" gate="1" x="35.56" y="182.88"/>
 <instance part="ADC7" gate="G$1" x="167.64" y="137.16" rot="R180"/>
 <instance part="ADC6" gate="G$1" x="167.64" y="124.46" rot="R180"/>
@@
 <instance part="+3V6" gate="G$1" x="33.02" y="7.62" rot="R270"/>
 <instance part="+3V7" gate="G$1" x="12.7" y="20.32" rot="R90"/>
+<instance part="R2" gate="G$1" x="15.24" y="195.58" rot="R180"/>
+<instance part="R3" gate="G$1" x="15.24" y="205.74" rot="R180"/>
+<instance part="R4" gate="G$1" x="15.24" y="185.42"/>
 </instances>
 <busses>
@@
 <pinref part="GREEN" gate="A" pin="A"/>
 <pinref part="GND10" gate="1" pin="GND"/>
-<wire x1="30.48" y1="185.42" x2="22.86" y2="185.42" width="0.1524" layer="91"/>
+<wire x1="35.56" y1="185.42" x2="27.94" y2="185.42" width="0.1524" layer="91"/>
 <pinref part="RED" gate="A" pin="A"/>
 <pinref part="YELLOW" gate="A" pin="A"/>
-<wire x1="22.86" y1="195.58" x2="22.86" y2="205.74" width="0.1524" layer="91"/>
-<wire x1="22.86" y1="195.58" x2="22.86" y2="185.42" width="0.1524" layer="91"/>
-<junction x="22.86" y="185.42"/>
-<junction x="22.86" y="195.58"/>
+<wire x1="27.94" y1="195.58" x2="27.94" y2="205.74" width="0.1524" layer="91"/>
+<wire x1="27.94" y1="195.58" x2="27.94" y2="185.42" width="0.1524" layer="91"/>
+<junction x="27.94" y="185.42"/>
+<junction x="27.94" y="195.58"/>
 </segment>
 <segment>
@@
 </segment>
 <segment>
-<pinref part="GREEN" gate="A" pin="K"/>
-<wire x1="7.62" y1="195.58" x2="7.62" y2="193.04" width="0.1524" layer="91"/>
-<wire x1="7.62" y1="193.04" x2="15.24" y2="185.42" width="0.1524" layer="91"/>
-<label x="10.16" y="185.42" size="1.778" layer="95"/>
+<label x="10.16" y="180.34" size="1.778" layer="95"/>
+<pinref part="R2" gate="G$1" pin="2"/>
+<wire x1="7.62" y1="195.58" x2="10.16" y2="195.58" width="0.1524" layer="91"/>
+<wire x1="7.62" y1="195.58" x2="7.62" y2="190.5" width="0.1524" layer="91"/>
+<pinref part="R4" gate="G$1" pin="1"/>
+<wire x1="7.62" y1="190.5" x2="10.16" y2="185.42" width="0.1524" layer="91"/>
 </segment>
 </net>
@@
 <label x="5.08" y="83.82" size="1.778" layer="95"/>
 </segment>
-<segment>
-<pinref part="YELLOW" gate="A" pin="K"/>
-<wire x1="7.62" y1="195.58" x2="15.24" y2="195.58" width="0.1524" layer="91"/>
-<label x="10.16" y="195.58" size="1.778" layer="95"/>
-</segment>
 </net>
 <net name="IO6" class="0">
@@
 </segment>
 <segment>
-<pinref part="RED" gate="A" pin="K"/>
-<wire x1="7.62" y1="195.58" x2="7.62" y2="198.12" width="0.1524" layer="91"/>
-<wire x1="7.62" y1="198.12" x2="15.24" y2="205.74" width="0.1524" layer="91"/>
-<label x="10.16" y="205.74" size="1.778" layer="95"/>
+<label x="10.16" y="208.28" size="1.778" layer="95"/>
+<pinref part="R3" gate="G$1" pin="2"/>
+<wire x1="7.62" y1="195.58" x2="7.62" y2="203.2" width="0.1524" layer="91"/>
+<wire x1="7.62" y1="203.2" x2="10.16" y2="205.74" width="0.1524" layer="91"/>
 </segment>
 </net>
@@
 </segment>
 </net>
+<net name="N$12" class="0">
+<segment>
+<pinref part="YELLOW" gate="A" pin="K"/>
+<pinref part="R2" gate="G$1" pin="1"/>
+</segment>
+</net>
+<net name="N$13" class="0">
+<segment>
+<pinref part="RED" gate="A" pin="K"/>
+<pinref part="R3" gate="G$1" pin="1"/>
+</segment>
+</net>
+<net name="N$14" class="0">
+<segment>
+<pinref part="R4" gate="G$1" pin="2"/>
+<pinref part="GREEN" gate="A" pin="K"/>
+</segment>
+</net>

Commit message: Fixed LED polarities, ADC power supplies
Connections:
- net +3V3: now also ADC4.2, ADC5.2, ADC6.2, ADC7.2
- net +5V: now also ADC0.2, ADC1.2, ADC2.2, ADC3.2, IC1.VREF
- net GND: now also GREEN.K, RED.K, YELLOW.K; no longer GREEN.A, RED.A, YELLOW.A
- net IO4: no longer R2.2
- net IO5: now also R2.2
- net N$12: now also GREEN.A, R4.2; no longer R2.1, YELLOW.K
- net N$13: now also R2.1, YELLOW.A; no longer R3.1, RED.K
- net N$14: now also R3.1, RED.A; no longer GREEN.K, R4.2
Other:
- moved on the sheet: GREEN, RED, YELLOW
Changed lines of the file:
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@@
 <part name="GND18" library="supply1" deviceset="GND" device=""/>
 <part name="GND19" library="supply1" deviceset="GND" device=""/>
-<part name="P+4" library="supply1" deviceset="+5V" device=""/>
-<part name="P+5" library="supply1" deviceset="+5V" device=""/>
-<part name="P+6" library="supply1" deviceset="+5V" device=""/>
-<part name="P+7" library="supply1" deviceset="+5V" device=""/>
 <part name="P+8" library="supply1" deviceset="+5V" device=""/>
-<part name="P+9" library="supply1" deviceset="+5V" device=""/>
-<part name="P+10" library="supply1" deviceset="+5V" device=""/>
-<part name="P+11" library="supply1" deviceset="+5V" device=""/>
 <part name="SV20" library="con-lstb" deviceset="MA03-1" device=""/>
 <part name="SV21" library="con-lstb" deviceset="MA03-1" device=""/>
@@
 <part name="R3" library="resistor" deviceset="R-US_" device="0309/V" value="10k"/>
 <part name="R4" library="resistor" deviceset="R-US_" device="0309/V" value="10k"/>
+<part name="P+4" library="supply1" deviceset="+5V" device=""/>
+<part name="P+5" library="supply1" deviceset="+5V" device=""/>
+<part name="P+6" library="supply1" deviceset="+5V" device=""/>
+<part name="+3V8" library="supply1" deviceset="+3V3" device=""/>
+<part name="+3V9" library="supply1" deviceset="+3V3" device=""/>
+<part name="+3V10" library="supply1" deviceset="+3V3" device=""/>
+<part name="+3V11" library="supply1" deviceset="+3V3" device=""/>
+<part name="P+7" library="supply1" deviceset="+5V" device=""/>
 </parts>
 <sheets>
@@
 <instance part="GND7" gate="1" x="78.74" y="114.3"/>
 <instance part="+3V5" gate="G$1" x="81.28" y="109.22" rot="R90"/>
-<instance part="GREEN" gate="A" x="22.86" y="185.42" rot="R270"/>
-<instance part="YELLOW" gate="A" x="22.86" y="195.58" rot="R270"/>
-<instance part="RED" gate="A" x="22.86" y="205.74" rot="R270"/>
+<instance part="GREEN" gate="A" x="30.48" y="185.42" rot="R90"/>
+<instance part="YELLOW" gate="A" x="30.48" y="195.58" rot="R90"/>
+<instance part="RED" gate="A" x="30.48" y="205.74" rot="R90"/>
 <instance part="GND10" gate="1" x="35.56" y="182.88"/>
 <instance part="ADC7" gate="G$1" x="167.64" y="137.16" rot="R180"/>
@@
 <instance part="GND18" gate="1" x="157.48" y="63.5" rot="R270"/>
 <instance part="GND19" gate="1" x="157.48" y="50.8" rot="R270"/>
-<instance part="P+4" gate="1" x="160.02" y="99.06" rot="R270"/>
-<instance part="P+5" gate="1" x="160.02" y="111.76" rot="R270"/>
-<instance part="P+6" gate="1" x="160.02" y="124.46" rot="R270"/>
-<instance part="P+7" gate="1" x="160.02" y="137.16" rot="R270"/>
-<instance part="P+8" gate="1" x="160.02" y="86.36" rot="R270"/>
-<instance part="P+9" gate="1" x="160.02" y="73.66" rot="R270"/>
-<instance part="P+10" gate="1" x="160.02" y="60.96" rot="R270"/>
-<instance part="P+11" gate="1" x="160.02" y="48.26" rot="R270"/>
+<instance part="P+8" gate="1" x="157.48" y="86.36" rot="R90"/>
 <instance part="SV20" gate="G$1" x="121.92" y="12.7" rot="R180"/>
 <instance part="SV21" gate="G$1" x="121.92" y="-2.54" rot="R180"/>
@@
 <instance part="R3" gate="G$1" x="15.24" y="205.74" rot="R180"/>
 <instance part="R4" gate="G$1" x="15.24" y="185.42"/>
+<instance part="P+4" gate="1" x="157.48" y="73.66" rot="R90"/>
+<instance part="P+5" gate="1" x="157.48" y="60.96" rot="R90"/>
+<instance part="P+6" gate="1" x="157.48" y="48.26" rot="R90"/>
+<instance part="+3V8" gate="G$1" x="157.48" y="99.06" rot="R90"/>
+<instance part="+3V9" gate="G$1" x="157.48" y="111.76" rot="R90"/>
+<instance part="+3V10" gate="G$1" x="157.48" y="124.46" rot="R90"/>
+<instance part="+3V11" gate="G$1" x="157.48" y="137.16" rot="R90"/>
+<instance part="P+7" gate="1" x="81.28" y="119.38" rot="R90"/>
 </instances>
 <busses>
@@
 </segment>
 <segment>
-<pinref part="GREEN" gate="A" pin="A"/>
-<pinref part="GND10" gate="1" pin="GND"/>
-<wire x1="35.56" y1="185.42" x2="27.94" y2="185.42" width="0.1524" layer="91"/>
-<pinref part="RED" gate="A" pin="A"/>
-<pinref part="YELLOW" gate="A" pin="A"/>
-<wire x1="27.94" y1="195.58" x2="27.94" y2="205.74" width="0.1524" layer="91"/>
-<wire x1="27.94" y1="195.58" x2="27.94" y2="185.42" width="0.1524" layer="91"/>
-<junction x="27.94" y="185.42"/>
-<junction x="27.94" y="195.58"/>
-</segment>
-<segment>
 <pinref part="ADC7" gate="G$1" pin="1"/>
 <pinref part="GND12" gate="1" pin="GND"/>
@@
 <pinref part="NEOPIXEL" gate="G$1" pin="1"/>
 <wire x1="48.26" y1="30.48" x2="58.42" y2="30.48" width="0.1524" layer="91"/>
+</segment>
+<segment>
+<pinref part="GND10" gate="1" pin="GND"/>
+<pinref part="GREEN" gate="A" pin="K"/>
+<wire x1="35.56" y1="185.42" x2="33.02" y2="185.42" width="0.1524" layer="91"/>
+<pinref part="YELLOW" gate="A" pin="K"/>
+<wire x1="33.02" y1="185.42" x2="33.02" y2="195.58" width="0.1524" layer="91"/>
+<pinref part="RED" gate="A" pin="K"/>
+<wire x1="33.02" y1="195.58" x2="33.02" y2="205.74" width="0.1524" layer="91"/>
+<junction x="33.02" y="195.58"/>
+<junction x="33.02" y="185.42"/>
 </segment>
 </net>
@@
 <pinref part="+3V7" gate="G$1" pin="+3V3"/>
 </segment>
+<segment>
+<pinref part="ADC4" gate="G$1" pin="2"/>
+<pinref part="+3V8" gate="G$1" pin="+3V3"/>
+</segment>
+<segment>
+<pinref part="ADC5" gate="G$1" pin="2"/>
+<pinref part="+3V9" gate="G$1" pin="+3V3"/>
+</segment>
+<segment>
+<pinref part="ADC6" gate="G$1" pin="2"/>
+<pinref part="+3V10" gate="G$1" pin="+3V3"/>
+</segment>
+<segment>
+<pinref part="ADC7" gate="G$1" pin="2"/>
+<pinref part="+3V11" gate="G$1" pin="+3V3"/>
+</segment>
 </net>
 <net name="!RESET" class="0">
@@
 <segment>
 <label x="10.16" y="180.34" size="1.778" layer="95"/>
-<pinref part="R2" gate="G$1" pin="2"/>
-<wire x1="7.62" y1="195.58" x2="10.16" y2="195.58" width="0.1524" layer="91"/>
 <wire x1="7.62" y1="195.58" x2="7.62" y2="190.5" width="0.1524" layer="91"/>
 <pinref part="R4" gate="G$1" pin="1"/>
@@
 <wire x1="2.54" y1="83.82" x2="22.86" y2="83.82" width="0.1524" layer="91"/>
 <label x="5.08" y="83.82" size="1.778" layer="95"/>
+</segment>
+<segment>
+<pinref part="R2" gate="G$1" pin="2"/>
+<wire x1="7.62" y1="195.58" x2="10.16" y2="195.58" width="0.1524" layer="91"/>
+<label x="10.16" y="198.12" size="1.778" layer="95"/>
 </segment>
 </net>
@@
 <pinref part="P+12" gate="1" pin="+5V"/>
 </segment>
+<segment>
+<pinref part="ADC3" gate="G$1" pin="2"/>
+<pinref part="P+8" gate="1" pin="+5V"/>
+</segment>
+<segment>
+<pinref part="ADC2" gate="G$1" pin="2"/>
+<pinref part="P+4" gate="1" pin="+5V"/>
+</segment>
+<segment>
+<pinref part="ADC1" gate="G$1" pin="2"/>
+<pinref part="P+5" gate="1" pin="+5V"/>
+</segment>
+<segment>
+<pinref part="ADC0" gate="G$1" pin="2"/>
+<pinref part="P+6" gate="1" pin="+5V"/>
+</segment>
+<segment>
+<pinref part="IC1" gate="G$1" pin="VREF"/>
+<pinref part="P+7" gate="1" pin="+5V"/>
+</segment>
 </net>
 <net name="DIO0" class="0">
@@
 <net name="N$12" class="0">
 <segment>
-<pinref part="YELLOW" gate="A" pin="K"/>
+<pinref part="R4" gate="G$1" pin="2"/>
+<pinref part="GREEN" gate="A" pin="A"/>
+<wire x1="25.4" y1="185.42" x2="20.32" y2="185.42" width="0.1524" layer="91"/>
+</segment>
+</net>
+<net name="N$13" class="0">
+<segment>
 <pinref part="R2" gate="G$1" pin="1"/>
-</segment>
-</net>
-<net name="N$13" class="0">
-<segment>
-<pinref part="RED" gate="A" pin="K"/>
+<pinref part="YELLOW" gate="A" pin="A"/>
+<wire x1="25.4" y1="195.58" x2="20.32" y2="195.58" width="0.1524" layer="91"/>
+</segment>
+</net>
+<net name="N$14" class="0">
+<segment>
 <pinref part="R3" gate="G$1" pin="1"/>
-</segment>
-</net>
-<net name="N$14" class="0">
-<segment>
-<pinref part="R4" gate="G$1" pin="2"/>
-<pinref part="GREEN" gate="A" pin="K"/>
-</segment>
-</net>
+<pinref part="RED" gate="A" pin="A"/>
+<wire x1="25.4" y1="205.74" x2="20.32" y2="205.74" width="0.1524" layer="91"/>
+</segment>
+</net>

Commit message: Some More Fun Connections
Lots of them. 32 actually.
Parts:
- removed SV24: (no value), con-lstb:MA03-1
- added IO10, IO11, IO12, IO13, IO14, IO15, IO16, IO17, IO18, IO19, IO20, IO21, IO22, IO23, IO24, IO25, IO26, IO27, IO28, IO29, IO30, IO31, IO5, IO6, IO7, IO8, IO9: (no value), con-lstb:MA03-1
- renumbered SV20 to SPI-CS, SV21 to SPI-CLK, SV22 to SPI-MOSI, SV23 to SPI-MISO, SV25 to IO4
Connections:
- net GND: now also IO20.1, IO31.1, IO4.1, IO5.1, IO6.1, IO7.1, SPI-CLK.1, SPI-CS.1, SPI-MISO.1, SPI-MOSI.1
- net IO13: now also IO13.3
- net N$10: now also ADC0.3
