File: projects/RoboRio/RoboRioExpansionBoard/ExpansionBoardV1.brd (EAGLE design)
At the start: 100.3 x 80.3 mm, 68 parts, among them IC1 MCP3008, Q1 5MHz

Commit message: Moved pin connections
LEDs moved to 16..18
Neopixel to 4
LCD to 5
Connections:
- net IO16: now also R4.1
- net IO17: now also R2.2
- net IO18: now also R3.2
- net IO4: now also LEVELSHIFTER.3; no longer R4.1
- net IO5: now also 3V3_LCD.3, LEVELSHIFTER.6; no longer R2.2
- net IO6: no longer R3.2
- net IO7: no longer LEVELSHIFTER.3
- net IO8: no longer 3V3_LCD.3, LEVELSHIFTER.6
Changed lines of the file:
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@@
 <signal name="IO4">
 <contactref element="PROPELLER" pad="5"/>
-<contactref element="R4" pad="1"/>
 <contactref element="IO4" pad="3"/>
-<wire x1="-66.04" y1="96.52" x2="67.31" y2="47.625" width="0" layer="19" extent="1-1"/>
-<wire x1="-93.98" y1="73.66" x2="-66.04" y2="96.52" width="0" layer="19" extent="1-1"/>
+<contactref element="LEVELSHIFTER" pad="3"/>
+<wire x1="-46.99" y1="2.54" x2="67.31" y2="47.625" width="0" layer="19" extent="1-1"/>
+<wire x1="-66.04" y1="96.52" x2="-46.99" y2="2.54" width="0" layer="19" extent="1-1"/>
 </signal>
 <signal name="IO5">
 <contactref element="PROPELLER" pad="6"/>
-<contactref element="R2" pad="2"/>
 <contactref element="IO5" pad="3"/>
-<wire x1="-76.2" y1="73.66" x2="67.31" y2="45.085" width="0" layer="19" extent="1-1"/>
-<wire x1="-76.2" y1="96.52" x2="-76.2" y2="73.66" width="0" layer="19" extent="1-1"/>
+<contactref element="LEVELSHIFTER" pad="6"/>
+<contactref element="3V3_LCD" pad="3"/>
+<wire x1="-35.56" y1="90.17" x2="67.31" y2="45.085" width="0" layer="19" extent="1-1"/>
+<wire x1="-76.2" y1="96.52" x2="-35.56" y2="90.17" width="0" layer="19" extent="1-1"/>
+<wire x1="-39.37" y1="2.54" x2="-35.56" y2="90.17" width="0" layer="19" extent="1-1"/>
 </signal>
 <signal name="IO6">
 <contactref element="PROPELLER" pad="7"/>
-<contactref element="R3" pad="2"/>
 <contactref element="IO6" pad="3"/>
-<wire x1="-83.82" y1="73.66" x2="67.31" y2="42.545" width="0" layer="19" extent="1-1"/>
-<wire x1="-86.36" y1="96.52" x2="-83.82" y2="73.66" width="0" layer="19" extent="1-1"/>
+<wire x1="-86.36" y1="96.52" x2="67.31" y2="42.545" width="0" layer="19" extent="1-1"/>
 </signal>
 <signal name="IO7">
 <contactref element="PROPELLER" pad="8"/>
-<contactref element="LEVELSHIFTER" pad="3"/>
 <contactref element="IO7" pad="3"/>
 <wire x1="-15.24" y1="102.87" x2="67.31" y2="40.005" width="0" layer="19" extent="1-1"/>
-<wire x1="-46.99" y1="2.54" x2="-15.24" y2="102.87" width="0" layer="19" extent="1-1"/>
 </signal>
 <signal name="IO8">
 <contactref element="PROPELLER" pad="13"/>
-<contactref element="LEVELSHIFTER" pad="6"/>
-<contactref element="3V3_LCD" pad="3"/>
 <contactref element="IO8" pad="3"/>
-<wire x1="-39.37" y1="2.54" x2="67.31" y2="27.305" width="0" layer="19" extent="1-1"/>
-<wire x1="-35.56" y1="90.17" x2="-39.37" y2="2.54" width="0" layer="19" extent="1-1"/>
-<wire x1="-25.4" y1="102.87" x2="-35.56" y2="90.17" width="0" layer="19" extent="1-1"/>
+<wire x1="-25.4" y1="102.87" x2="67.31" y2="27.305" width="0" layer="19" extent="1-1"/>
 </signal>
 <signal name="IO9">
@@
 <contactref element="PROPELLER" pad="21"/>
 <contactref element="IO16" pad="3"/>
+<contactref element="R4" pad="1"/>
 <wire x1="82.55" y1="9.525" x2="90.17" y2="10.16" width="0" layer="19" extent="1-1"/>
+<wire x1="-93.98" y1="73.66" x2="82.55" y2="9.525" width="0" layer="19" extent="1-1"/>
 </signal>
 <signal name="IO17">
 <contactref element="PROPELLER" pad="22"/>
 <contactref element="IO17" pad="3"/>
+<contactref element="R2" pad="2"/>
 <wire x1="82.55" y1="12.065" x2="90.17" y2="12.7" width="0" layer="19" extent="1-1"/>
+<wire x1="-76.2" y1="73.66" x2="82.55" y2="12.065" width="0" layer="19" extent="1-1"/>
 </signal>
 <signal name="IO18">
 <contactref element="PROPELLER" pad="23"/>
 <contactref element="IO18" pad="3"/>
+<contactref element="R3" pad="2"/>
 <wire x1="82.55" y1="14.605" x2="90.17" y2="15.24" width="0" layer="19" extent="1-1"/>
+<wire x1="-83.82" y1="73.66" x2="82.55" y2="14.605" width="0" layer="19" extent="1-1"/>
 </signal>
 <signal name="IO19">
